File: hardware/src/LEDx11.kicad_sch (KiCad schematic)
At the start: 22 parts

Commit message: Add: RTC schematic
Parts:
- renumbered D801 to D701
Changed lines of the file:
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@@
 		(dnp no)
 		(fields_autoplaced yes)
-		(property "Reference" "D801"
+		(property "Reference" "D701"
 			(at 113.03 44.4814 0)
 			(effects

Commit message: Mod: RTC GPIOs
Parts:
- renumbered C701 to C801, C702 to C802, C703 to C803, C704 to C804, C705 to C805, C706 to C806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
