File: hardware/src/LEDx4.kicad_sch (KiCad schematic)
At the start: 8 parts

Commit message: Mod: RTC GPIOs
Parts:
- renumbered C719 to C701, C720 to C702, C721 to C703, C722 to C704, D712 to D701, D715 to D702, D718 to D703, D721 to D704
Changed lines of the file:
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@@
 		(dnp no)
 		(fields_autoplaced yes)
-		(property "Reference" "#PWR0756"
+		(property "Reference" "#PWR0702"
 			(at 101.6 67.31 0)
 			(effects
@@
 			(project "ESP-Wordclock"
 				(path "/bfaac094-0365-40a4-8b7a-d4d62ace544e/c23f8616-5eaa-4df3-8ee0-2a2271a82cce/ba4e66ee-1ea7-408a-a977-ad0048349e9f"
-					(reference "#PWR0756")
+					(reference "#PWR0702")
 					(unit 1)
 				)
@@
 		(dnp no)
 		(fields_autoplaced yes)
-		(property "Reference" "#PWR0774"
+		(property "Reference" "#PWR0708"
 			(at 139.7 190.5 0)
 			(effects
@@
 			(project "ESP-Wordclock"
 				(path "/bfaac094-0365-40a4-8b7a-d4d62ace544e/c23f8616-5eaa-4df3-8ee0-2a2271a82cce/ba4e66ee-1ea7-408a-a977-ad0048349e9f"
-					(reference "#PWR0774")
+					(reference "#PWR0708")
 					(unit 1)
 				)
@@
 		(dnp no)
 		(fields_autoplaced yes)
-		(property "Reference" "#PWR0785"
+		(property "Reference" "#PWR0715"
 			(at 177.8 44.45 0)
 			(effects
@@
 			(project "ESP-Wordclock"
 				(path "/bfaac094-0365-40a4-8b7a-d4d62ace544e/c23f8616-5eaa-4df3-8ee0-2a2271a82cce/ba4e66ee-1ea7-408a-a977-ad0048349e9f"
-					(reference "#PWR0785")
+					(reference "#PWR0715")
 					(unit 1)
 				)
@@
 		(dnp no)
 		(fields_autoplaced yes)
-		(property "Reference" "C719"
+		(property "Reference" "C701"
 			(at 130.81 176.5299 0)
 			(effects
@@
 			(project "ESP-Wordclock"
 				(path "/bfaac094-0365-40a4-8b7a-d4d62ace544e/c23f8616-5eaa-4df3-8ee0-2a2271a82cce/ba4e66ee-1ea7-408a-a977-ad0048349e9f"
-					(reference "C719")
+					(reference "C701")
 					(unit 1)
 				)
@@
 		(dnp no)
 		(fields_autoplaced yes)
-		(property "Reference" "#PWR0776"
+		(property "Reference" "#PWR0710"
 			(at 152.4 67.31 0)
 			(effects
@@
 			(project "ESP-Wordclock"
 				(path "/bfaac094-0365-40a4-8b7a-d4d62ace544e/c23f8616-5eaa-4df3-8ee0-2a2271a82cce/ba4e66ee-1ea7-408a-a977-ad0048349e9f"
-					(reference "#PWR0776")
+					(reference "#PWR0710")
 					(unit 1)
 				)
@@
 		(dnp no)
 		(fields_autoplaced yes)
-		(property "Reference" "#PWR0765"
+		(property "Reference" "#PWR0703"
 			(at 127 44.45 0)
 			(effects
@@
 			(project "ESP-Wordclock"
 				(path "/bfaac094-0365-40a4-8b7a-d4d62ace544e/c23f8616-5eaa-4df3-8ee0-2a2271a82cce/ba4e66ee-1ea7-408a-a977-ad0048349e9f"
-					(reference "#PWR0765")
+					(reference "#PWR0703")
 					(unit 1)
 				)
@@
 		(dnp no)
 		(fields_autoplaced yes)
-		(property "Reference" "#PWR0786"
+		(property "Reference" "#PWR0716"
 			(at 177.8 67.31 0)
 			(effects
@@
 			(project "ESP-Wordclock"
 				(path "/bfaac094-0365-40a4-8b7a-d4d62ace544e/c23f8616-5eaa-4df3-8ee0-2a2271a82cce/ba4e66ee-1ea7-408a-a977-ad0048349e9f"
-					(reference "#PWR0786")
+					(reference "#PWR0716")
 					(unit 1)
 				)
@@
 		(dnp no)
 		(fields_autoplaced yes)
-		(property "Reference" "#PWR0755"
+		(property "Reference" "#PWR0701"
 			(at 101.6 44.45 0)
 			(effects
@@
 			(project "ESP-Wordclock"
 				(path "/bfaac094-0365-40a4-8b7a-d4d62ace544e/c23f8616-5eaa-4df3-8ee0-2a2271a82cce/ba4e66ee-1ea7-408a-a977-ad0048349e9f"
-					(reference "#PWR0755")
+					(reference "#PWR0701")
 					(unit 1)
 				)
@@
 		(dnp no)
 		(fields_autoplaced yes)
-		(property "Reference" "C720"
+		(property "Reference" "C702"
 			(at 143.51 176.5299 0)
 			(effects
@@
 			(project "ESP-Wordclock"
 				(path "/bfaac094-0365-40a4-8b7a-d4d62ace544e/c23f8616-5eaa-4df3-8ee0-2a2271a82cce/ba4e66ee-1ea7-408a-a977-ad0048349e9f"
-					(reference "C720")
+					(reference "C702")
 					(unit 1)
 				)
@@
 		(dnp no)
 		(fields_autoplaced yes)
-		(property "Reference" "D715"
+		(property "Reference" "D702"
 			(at 138.43 44.4814 0)
 			(effects
@@
 			(project "ESP-Wordclock"
 				(path "/bfaac094-0365-40a4-8b7a-d4d62ace544e/c23f8616-5eaa-4df3-8ee0-2a2271a82cce/ba4e66ee-1ea7-408a-a977-ad0048349e9f"
-					(reference "D715")
+					(reference "D702")
 					(unit 1)
 				)
@@
 		(dnp no)
 		(fields_autoplaced yes)
-		(property "Reference" "#PWR0781"
+		(property "Reference" "#PWR0711"
 			(at 152.4 175.26 0)
 			(effects
@@
 			(project "ESP-Wordclock"
 				(path "/bfaac094-0365-40a4-8b7a-d4d62ace544e/c23f8616-5eaa-4df3-8ee0-2a2271a82cce/ba4e66ee-1ea7-408a-a977-ad0048349e9f"
-					(reference "#PWR0781")
+					(reference "#PWR0711")
 					(unit 1)
 				)
@@
 		(dnp no)
 		(fields_autoplaced yes)
-		(property "Reference" "#PWR0771"
+		(property "Reference" "#PWR0705"
 			(at 127 175.26 0)
 			(effects
@@
 			(project "ESP-Wordclock"
 				(path "/bfaac094-0365-40a4-8b7a-d4d62ace544e/c23f8616-5eaa-4df3-8ee0-2a2271a82cce/ba4e66ee-1ea7-408a-a977-ad0048349e9f"
-					(reference "#PWR0771")
+					(reference "#PWR0705")
 					(unit 1)
 				)
@@
 		(dnp no)
 		(fields_autoplaced yes)
-		(property "Reference" "D721"
+		(property "Reference" "D704"
 			(at 189.23 44.4814 0)
 			(effects
@@
 			(project "ESP-Wordclock"
 				(path "/bfaac094-0365-40a4-8b7a-d4d62ace544e/c23f8616-5eaa-4df3-8ee0-2a2271a82cce/ba4e66ee-1ea7-408a-a977-ad0048349e9f"
-					(reference "D721")
+					(reference "D704")
 					(unit 1)
 				)
@@
 		(dnp no)
 		(fields_autoplaced yes)
-		(property "Reference" "#PWR0772"
+		(property "Reference" "#PWR0706"
 			(at 127 190.5 0)
 			(effects
@@
 			(project "ESP-Wordclock"
 				(path "/bfaac094-0365-40a4-8b7a-d4d62ace544e/c23f8616-5eaa-4df3-8ee0-2a2271a82cce/ba4e66ee-1ea7-408a-a977-ad0048349e9f"
-					(reference "#PWR0772")
+					(reference "#PWR0706")
 					(unit 1)
 				)
@@
 		(dnp no)
 		(fields_autoplaced yes)
-		(property "Reference" "#PWR0773"
+		(property "Reference" "#PWR0707"
 			(at 139.7 175.26 0)
 			(effects
@@
 			(project "ESP-Wordclock"
 				(path "/bfaac094-0365-40a4-8b7a-d4d62ace544e/c23f8616-5eaa-4df3-8ee0-2a2271a82cce/ba4e66ee-1ea7-408a-a977-ad0048349e9f"
-					(reference "#PWR0773")
+					(reference "#PWR0707")
 					(unit 1)
 				)
@@
 		(dnp no)
 		(fields_autoplaced yes)
-		(property "Reference" "#PWR0784"
+		(property "Reference" "#PWR0714"
 			(at 165.1 190.5 0)
 			(effects
@@
 			(project "ESP-Wordclock"
 				(path "/bfaac094-0365-40a4-8b7a-d4d62ace544e/c23f8616-5eaa-4df3-8ee0-2a2271a82cce/ba4e66ee-1ea7-408a-a977-ad0048349e9f"
-					(reference "#PWR0784")
+					(reference "#PWR0714")
 					(unit 1)
 				)
@@
 		(dnp no)
 		(fields_autoplaced yes)
-		(property "Reference" "D712"
+		(property "Reference" "D701"
 			(at 113.03 44.4814 0)
 			(effects
@@
 			(project "ESP-Wordclock"
 				(path "/bfaac094-0365-40a4-8b7a-d4d62ace544e/c23f8616-5eaa-4df3-8ee0-2a2271a82cce/ba4e66ee-1ea7-408a-a977-ad0048349e9f"
-					(reference "D712")
+					(reference "D701")
 					(unit 1)
 				)
@@
 		(dnp no)
 		(fields_autoplaced yes)
-		(property "Reference" "#PWR0783"
+		(property "Reference" "#PWR0713"
 			(at 165.1 175.26 0)
 			(effects
@@
 			(project "ESP-Wordclock"
 				(path "/bfaac094-0365-40a4-8b7a-d4d62ace544e/c23f8616-5eaa-4df3-8ee0-2a2271a82cce/ba4e66ee-1ea7-408a-a977-ad0048349e9f"
-					(reference "#PWR0783")
+					(reference "#PWR0713")
 					(unit 1)
 				)
@@
 		(dnp no)
 		(fields_autoplaced yes)
-		(property "Reference" "#PWR0775"
+		(property "Reference" "#PWR0709"
 			(at 152.4 44.45 0)
 			(effects
@@
 			(project "ESP-Wordclock"
 				(path "/bfaac094-0365-40a4-8b7a-d4d62ace544e/c23f8616-5eaa-4df3-8ee0-2a2271a82cce/ba4e66ee-1ea7-408a-a977-ad0048349e9f"
-					(reference "#PWR0775")
+					(reference "#PWR0709")
 					(unit 1)
 				)
@@
 		(dnp no)
 		(fields_autoplaced yes)
-		(property "Reference" "#PWR0782"
+		(property "Reference" "#PWR0712"
 			(at 152.4 190.5 0)
 			(effects
@@
 			(project "ESP-Wordclock"
 				(path "/bfaac094-0365-40a4-8b7a-d4d62ace544e/c23f8616-5eaa-4df3-8ee0-2a2271a82cce/ba4e66ee-1ea7-408a-a977-ad0048349e9f"
-					(reference "#PWR0782")
+					(reference "#PWR0712")
 					(unit 1)
 				)
@@
 		(dnp no)
 		(fields_autoplaced yes)
-		(property "Reference" "C721"
+		(property "Reference" "C703"
 			(at 156.21 176.5299 0)
 			(effects
@@
 			(project "ESP-Wordclock"
 				(path "/bfaac094-0365-40a4-8b7a-d4d62ace544e/c23f8616-5eaa-4df3-8ee0-2a2271a82cce/ba4e66ee-1ea7-408a-a977-ad0048349e9f"
-					(reference "C721")
+					(reference "C703")
 					(unit 1)
 				)
@@
 		(dnp no)
 		(fields_autoplaced yes)
-		(property "Reference" "C722"
+		(property "Reference" "C704"
 			(at 168.91 176.5299 0)
 			(effects
@@
 			(project "ESP-Wordclock"
 				(path "/bfaac094-0365-40a4-8b7a-d4d62ace544e/c23f8616-5eaa-4df3-8ee0-2a2271a82cce/ba4e66ee-1ea7-408a-a977-ad0048349e9f"
-					(reference "C722")
+					(reference "C704")
 					(unit 1)
 				)
@@
 		(dnp no)
 		(fields_autoplaced yes)
-		(property "Reference" "D718"
+		(property "Reference" "D703"
 			(at 163.83 44.4814 0)
 			(effects
@@
 			(project "ESP-Wordclock"
 				(path "/bfaac094-0365-40a4-8b7a-d4d62ace544e/c23f8616-5eaa-4df3-8ee0-2a2271a82cce/ba4e66ee-1ea7-408a-a977-ad0048349e9f"
-					(reference "D718")
+					(reference "D703")
 					(unit 1)
 				)
@@
 		(dnp no)
 		(fields_autoplaced yes)
-		(property "Reference" "#PWR0766"
+		(property "Reference" "#PWR0704"
 			(at 127 67.31 0)
 			(effects
@@
 			(project "ESP-Wordclock"
 				(path "/bfaac094-0365-40a4-8b7a-d4d62ace544e/c23f8616-5eaa-4df3-8ee0-2a2271a82cce/ba4e66ee-1ea7-408a-a977-ad0048349e9f"
-					(reference "#PWR0766")
-					(unit 1)
-				)
+					(reference "#PWR0704")
+					(unit 1)
+				)
